File: amp.kicad_sch (KiCad schematic)
At the start: 85 parts, among them J1 Screw_Terminal_01x02, J2 Screw_Terminal_01x02, J3 Screw_Terminal_01x02, J4 Screw_Terminal_01x02, J5 Screw_Terminal_01x02, J6 state, J7 Preamp, Q1 2N7002, Q2 2N7002, U1 7812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

Commit message: schematic annotations
Other:
- note added: "F_{PWM} = 600kHz"
- note added: "LM4040BIM3-5.0 60uA < i_{z} < 15mA R_{s}=10k i_{z}=0.7mA"
- note removed: "LM4040BIM3-5.0 60uA < i_{z} < 15mA R=10k i_{z}=0.7mA"
Changed lines of the file:
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@@
 	)
 	(image
-		(at 153.289 149.606)
+		(at 213.487 70.612)
 		(scale 0.189333)
 		(data "iVBORw0KGgoAAAANSUhEUgAABxAAAAQeCAIAAAB37zjWAAAAA3NCSVQICAjb4U/gAAAACXBIWXMA"
@@
 	(text "00 = stereo BTL"
 		(exclude_from_sim no)
-		(at 431.546 211.582 0)
+		(at 428.498 210.312 0)
 		(effects
 			(font
@@
 		)
 	)
-	(text "LM4040BIM3-5.0\n60uA < i_{z} < 15mA\nR=10k i_{z}=0.7mA"
+	(text "LM4040BIM3-5.0\n60uA < i_{z} < 15mA\nR_{s}=10k i_{z}=0.7mA"
 		(exclude_from_sim no)
 		(at 150.622 80.518 0)
@@
 		)
 	)
+	(text "F_{PWM} = 600kHz"
+		(exclude_from_sim no)
+		(at 429.768 149.86 0)
+		(effects
+			(font
+				(size 1.27 1.27)
+			)
+		)
+	)
